Commit message: Implementação e simulação sensor ultrassonico, bem como flexbe

File: ros/rqt/ros_ws/src/ros_robotics/urdf/rrbot.xacro (robot description, xacro)
@@ -89,5 +89,5 @@
       <origin xyz="0 0 ${height3/2 - axle_offset}" rpy="0 0 0"/>
       <geometry>
-	<box size="${width} ${width} ${height3}"/>
+	    <box size="${width} ${width} ${height3}"/>
       </geometry>
       <material name="blue"/>
@@ -96,8 +96,33 @@
       <origin xyz="0 0 ${height3/2 - axle_offset}" rpy="0 0 0"/>
       <geometry>
-	<box size="${width} ${width} ${height3}"/>
+	    <box size="${width} ${width} ${height3}"/>
       </geometry>
     </collision>
     <xacro:default_inertial z_value="${height3/2 - axle_offset}" i_value="1.0" mass="1"/>
+  </link>
+  <joint name="sensor_ultrasonic_joint" type="fixed">
+    <axis xyz="0 1 0" />
+    <origin rpy="0 0 0" xyz="0 0 ${height3}" />
+    <parent link="top_link"/>
+    <child link="sensor_ultrasonic_link"/>
+  </joint>
+  <link name="sensor_ultrasonic_link">
+      <visual>
+        <origin xyz="0 0 0" rpy="0 0 0"/>
+        <geometry>
+          <box size="0.02 0.02 0.02"/>
+        </geometry>
+      </visual>
+      <collision>
+        <origin xyz="0 0 0" rpy="0 0 0"/>
+        <geometry>
+          <box size="0.02 0.02 0.02"/>
+        </geometry>
+      </collision>
+      <inertial>
+        <mass value="1e-5" />
+        <origin xyz="0 0 0" rpy="0 0 0"/>
+        <inertia ixx="1e-6" ixy="0" ixz="0" iyy="1e-6" iyz="0" izz="1e-6" />
+      </inertial>
   </link>
   <transmission name="transmission1">
